File: MPPTBatteryCharger/MPPTBatteryCharger.brd (EAGLE design)
At the start: 45.7 x 21.6 mm, 64 parts, among them J1 2S-BATTERYSMD, Q1 DMN6040SSD-13, Q2 DMN6040SSD-13, Q3 220mA/50V/3.5Ω, U1 BQ24650, U2 BQ28Z610

Commit message: As per Dec 2019 board orders
Parts:
- removed TP3, TP4, TP5: TPPAD1-13Y, testpad:P1-13Y
- removed TS: STRAWSON_EAGLE_LIB_JST_SH_4, BeagleBone_Blue:STRAWSON_EAGLE_LIB_JST_SH_4_SMD
- added BAL, BAT, RET: TPPAD1-13Y, testpad:P1-13Y
- added C15: 1u, resistor:C0402
- added C16: 10n, resistor:C0402
- added C17, C19, C20: 100n, resistor:C0402
- added C18: 2u2, resistor:C0603
- added H2: MOUNT-PAD-ROUND2.8, holes:2,8-PAD
- added JP3: (no value), pinhead:1X10
- added Q4, Q5: AO3400A, PowerComponents:SOT23
- added Q6: AO3400A, SparkFun-DiscreteSemi:SOT23-3
- added R28: 330R, resistor:R0402
- added R29: 10K, resistor:R0402
- added U3: HY2213, PowerComponents:SOT23-6L
- added U4: BQ24650, PowerComponents:QFN16
- added U5: R5460X2XX, PowerComponents:SOT23-6L
- C1: value 2u2 -> 10u; device resistor:C0603 -> resistor:C1206
- C10, C14, C7: device resistor:C0603 -> resistor:C0402
- C11: value 22p -> 10u; device resistor:C0603 -> resistor:C1206
- C12: value 2u2 -> 100n; device resistor:C0603 -> resistor:C0402
- C13: value 100n -> 1u; device resistor:C0603 -> resistor:C0402
- C2, C3, C8: value 10u -> 100n; device resistor:C1210 -> resistor:C0402
- C4: value 1u -> 100n; device resistor:C0603 -> resistor:C0402
- C5: value 1u -> 10u; device resistor:C0603 -> resistor:C1206
- C6: value 100n -> 4u7; device resistor:C0603 -> resistor:C1206
- C9: value 4u7 -> 22p; device resistor:C1210 -> resistor:C0402
- D2: value 700mA/40V/533mV -> BAS70-04
- JP1: device pinhead:1X10 -> pinhead:1X03
- L1: device PowerComponents:DG6050 -> PowerComponents:MWSA1205
- Q1: value DMN6040SSD-13 -> FS8205; device transistor-power:SO-08 -> PowerComponents:SOT23-6L
- Q2: value DMN6040SSD-13 -> AO3400A; device transistor-power:SO-08 -> PowerComponents:SOT23
- Q3: value 220mA/50V/3.5Ω -> AO3400A; device SparkFun-DiscreteSemi:SOT23-3 -> PowerComponents:SOT23
- R1: value 2R -> 5K1; device resistor:R0603 -> resistor:R0402
- R10: value 10R -> 4R7
- R11: value 40m -> 20K; device resistor:R2512 -> resistor:R0402
- R12: value 100K -> 300K; device resistor:R0603 -> resistor:R0402
- R13, R19, R20, R21, R26: device resistor:R0603 -> resistor:R0402
- R14: value 10K -> 2R; device resistor:R0603 -> resistor:R1206
- R15: value 10K -> 1K5; device resistor:R0603 -> resistor:R0402
- R16: value 300K -> 10K
- R17: value 2m -> 82K; device resistor:R2512 -> resistor:R0603
- R18: value 100R -> 1K; device resistor:R0603 -> resistor:R0402
- R2: value (none) -> 5K1; device resistor:R0603 -> resistor:R0402
- R22: value 10M -> 10K; device resistor:R0603 -> resistor:R0402
- R23: value 5K1 -> 27K; device resistor:R0603 -> resistor:R0402
- R24: value 5K1 -> 4K7; device resistor:R0603 -> resistor:R0402
- R25: value 10M -> 330R; device resistor:R0603 -> resistor:R0402
- R27: value 5R -> 10K; device resistor:R0603 -> resistor:R0402
- R3: value (none) -> 100R; device resistor:R0603 -> resistor:R0402
- R4: value 232K -> 0R02; device resistor:R0603 -> resistor:R1206
- R5: value 15K -> 100R; device resistor:R0603 -> resistor:R0402
- R6: value 100R -> 0R016; device resistor:R0603 -> resistor:R1206
- R7: value 10K -> 100R; device resistor:R0603 -> resistor:R0402
- R8: value 5K1 -> 4R7; device resistor:R0603 -> resistor:R1206
- R9: value 5K1 -> 100K; device resistor:R0603 -> resistor:R0402
- U1: value BQ24650 -> HY2213; device PowerComponents:QFN16 -> PowerComponents:SOT23-6L
- U2: value BQ28Z610 -> BQ34Z100-G1; device PowerComponents:PDSO-N12 -> PowerComponents:TSSOP14
- moved R10 49.6 mm to (58.3, 12.1), turned to 0 degrees
- moved R4 48.7 mm to (54.6, 19.7), flipped to the top, turned to 270 degrees
- moved Q3 47.4 mm to (53.3, 15.2), flipped to the top
- moved R3 45.9 mm to (52.1, 21.0), flipped to the top
- moved R5 45.9 mm to (52.1, 19.1), flipped to the top
- moved Q1 42.0 mm to (58.4, 19.7), turned to 0 degrees
- moved H1 40.9 mm to (3.17, 22.2)
- moved R7 40.9 mm to (47.0, 15.9), flipped to the top, turned to 270 degrees
- moved C2 40.3 mm to (47.0, 21.0), turned to 0 degrees
- moved U1 39.4 mm to (49.5, 15.9), flipped to the top
- moved C4 39.3 mm to (49.5, 19.1), flipped to the top, turned to 0 degrees
- moved C3 39.1 mm to (49.5, 21.0), turned to 0 degrees
- moved JP2 37.7 mm to (55.9, 24.1), turned to 0 degrees
- moved C7 37.4 mm to (45.1, 15.9), flipped to the top, turned to 90 degrees
- moved R1 36.8 mm to (39.4, 21.0)
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- renumbered TP1 to P-, TP2 to P+
Connections:
- removed net BAT: J1.BAT, Q2.1, R25.2, R27.1, TP4.TP
- removed net CHG_GATE: R24.1, U2.9
- removed net DSG_GATE: R23.1, U2.7
- removed net N$32: C13.1, C14.1, R26.2, U2.12
- removed net N$33: C14.2, R27.2, U2.11
- removed net N$34: C12.1, U2.10
- removed net N$37: C10.1, R13.1, U2.2
- removed net N$39: C10.2, R18.1, U2.3
- new net N$13: Q3.1, U1.6
- new net N$15: Q3.3, R8.1
- new net N$16: R16.2, R17.1, U2.4
- new net N$2: Q5.1, U3.6
- new net N$20: C10.1, R13.1, U3.2
- new net N$21: C7.1, R7.1, U1.2
- new net N$22: R18.1, U5.3
- new net N$23: C19.1, R25.2, U5.4
- new net N$24: C20.1, R28.1, U5.5
- new net N$27: Q1.4, U5.1
- new net N$29: C2.1, C3.2, R3.2, U2.9
- new net N$30: C12.1, U2.6
- new net REG25: C13.1, JP1.2, U2.7
- new net STAT_LED_EN: JP3.5, STAT1.A, STAT2.A
- net !BAT_CE!: now also JP3.3, R26.1; no longer JP1.4, R6.1
- net +3V3: now also JP2.1, R1.2, R2.2; no longer JP1.1, R8.2, R9.2, STAT1.A, STAT2.A
- net AGND: now also C12.2, C13.2, C14.2, Q6.2, R15.1, R16.1, R20.1, R23.1, R9.1, U2.1, U2.12, U2.2, U2.3, U2.8; no longer C4.2, Q3.2, R12.1, R3.1, R5.1, R7.1, TS.1, TS.3
- net BAL: now also BAL.TP, C10.2, Q5.2, R25.1, R7.2, R8.2, U3.3; no longer R26.1, TP5.TP
- net GND: now also C11.2, C15.2, C18.2, C3.1, C4.1, C6.2, H2.B2,8, JP3.10, JP3.6, JP3.7, JP3.8, JP3.9, Q2.2, R22.1, R29.1, R3.1, R4.1, U4.11, U4.TH; no longer C12.2, C13.2, C2.2, C3.2, C8.2, C9.2, JP2.10, JP2.5, JP2.6, JP2.7, JP2.8, JP2.9, Q1.1, R14.1, R15.1, R17.2, R18.2, U1.11, U1.TH, U2.1, U2.EP, U2.EP1, U2.EP2, U2.EP3, U2.EP4
- net MPPSET: now also Q6.3, R11.1, R15.2, U4.2; no longer Q3.3, R4.1, R5.2, U1.2
- net N$1: now also C18.1, R14.1; no longer C1.1, R1.1
- net N$10: now also C17.1, U4.16; no longer C7.1, U1.16
- net N$11: now also C15.1, U4.12; no longer C5.1, U1.12
- net N$12: now also C9.2, R12.1, R9.2, U4.8; no longer C11.2, R12.2, R16.1, U1.8
- net N$14: now also R21.1; no longer R20.1
- net N$18: now also Q5.3, R10.1; no longer R19.1, U2.8
- net N$25: now also C16.1, Q1.1, R18.2, R4.2, R5.1; no longer Q2.5, Q2.6, Q2.7, Q2.8
- net N$26: now also Q1.6, U5.2; no longer Q2.4, R22.1, R23.2
- net N$28: now also C2.2, C4.2, R5.2, U2.10; no longer Q2.2, R24.2, R25.1
- net N$3: now also R19.2, U4.1; no longer R10.2, U1.1
- net N$4: now also C11.1, C5.1, Q4.3, R11.2, R19.1; no longer C2.1, C3.1, Q1.5, Q1.6, R10.1, R4.2
- net N$47: now also R27.1; no longer R21.1
- net N$5: now also Q4.1, U4.15; no longer Q1.4, U1.15
- net N$6: now also C17.2, Q2.3, Q4.2, U4.14; no longer C7.2, Q1.3, Q1.7, Q1.8, U1.14
- net N$7: now also Q2.1, U4.13; no longer Q1.2, U1.13
- net N$8: now also Q6.1, R20.2, R26.2; no longer Q3.1, R6.2, R7.2
- net N$81: now also R29.2; no longer R14.2
- net N$83: now also R22.2; no longer R15.2
- net N$9: now also C8.1, R6.1, U4.10; no longer C6.1, R11.1, U1.10
- net PANEL: now also JP3.4, R14.2; no longer JP2.3, R1.2
- net RET: now also C16.2, C19.2, C20.2, C7.2, Q1.3, Q3.2, RET.TP, U1.3, U5.6; no longer R13.2, R17.1, TP3.TP
- net SCL: now also JP2.3, R2.1, U2.13; no longer JP2.2, R9.1, U2.5
- net SDA: now also JP2.2, R1.1, U2.14; no longer JP2.1, R8.1, U2.6
- net STAT1: now also JP3.1, R21.2, U4.3; no longer JP1.2, R20.2, U1.3
- net STAT2: now also JP3.2, R27.2, U4.5; no longer JP1.3, R21.2, U1.5
- net TS1: now also JP1.3, R23.2, R24.1, U4.4; no longer R2.1, R3.2, TS.2, U1.4
- net TS2: now also JP1.1, U2.11; no longer TS.4, U2.4
- net VBAT: now also BAT.TP, C1.1, C6.1, C8.2, J1.BAT, JP2.10, JP2.5, JP2.6, JP2.7, JP2.8, JP2.9, R10.2, R12.2, R13.2, R17.2, R28.2, R6.2, U4.9; no longer C11.1, C6.2, C8.1, JP1.10, JP1.5, JP1.6, JP1.7, JP1.8, JP1.9, Q2.3, R11.2, R16.2, R19.2, R22.2, U1.9
- net VREF: now also C14.1, R24.2, U4.6, U4.7; no longer C4.1, R2.2, U1.6, U1.7
Routing:
- net +3V3: track 63.6 -> 6.13 mm, vias 2 -> 0
- net VBAT: track 65.8 -> 123.1 mm, vias 3 -> 4
- net RET: track 15.3 -> 60.2 mm, vias 1 -> 5
- net VREF: track 8.08 -> 36.8 mm, vias 0 -> 3
- net REG25: track 0.00 -> 24.9 mm, vias 0 -> 2
- net BAL: track 29.6 -> 50.4 mm, vias 1 -> 2
- net BAT: track 20.4 -> 0.00 mm, vias 2 -> 0
- net MPPSET: track 9.03 -> 27.1 mm, vias 0 -> 3
- net N$25: track 3.81 -> 20.1 mm, vias 0 -> 2
- net N$27: track 0.00 -> 13.6 mm, vias 0 -> 2
- net DSG_GATE: track 13.2 -> 0.00 mm, vias 2 -> 0
- net N$39: track 12.8 -> 0.00 mm, vias 2 -> 0
- net CHG_GATE: track 12.4 -> 0.00 mm, vias 2 -> 0
- net N$11: track 4.66 -> 16.9 mm, vias 0 -> 4
- net N$29: track 0.00 -> 11.9 mm
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- added copper zone on layer 15, net AGND
- added copper zone on layer 2, net GND
- removed copper zone on layer 2, net AGND
- removed copper zone on layer 15, net GND
Other:
- board size 45.7 x 21.6 mm -> 73 x 25.4 mm
- board text added: "P+"
- board text added: "P-"
- board text added: "Project Ladon Battery Charger Rev A -- 2019 Oct 15"
- board text removed: "PANEL1+"
- board text removed: "PANEL1-"
