File: MPPTBatteryCharger/MPPTBatteryCharger.sch (EAGLE design)
At the start: 64 parts, among them J1 2S-BATTERYSMD, Q1 DMN6040SSD-13, Q2 DMN6040SSD-13, Q3 220mA/50V/3.5Ω, U1 BQ24650, U2 BQ28Z610

Commit message: As per Dec 2019 board orders
Parts:
- removed TP1, TP2, TP3, TP4, TP5: TPPAD1-13Y, testpad:TPPAD1-13Y
- removed TS: STRAWSON_EAGLE_LIB_JST_SH_4, BeagleBone_Blue:STRAWSON_EAGLE_LIB_JST_SH_4
- added BAL, BAT, P+, P-, RET: TPPAD1-13Y, testpad:TPPAD1-13Y
- added C15: 1u, resistor:C-EUC0402
- added C16: 10n, resistor:C-EUC0402
- added C17, C19, C20: 100n, resistor:C-EUC0402
- added C18: 2u2, resistor:C-EUC0603
- added H2: MOUNT-PAD-ROUND2.8, holes:MOUNT-PAD-ROUND2.8
- added JP3: (no value), pinhead:PINHD-1X10
- added Q4, Q5: AO3400A, PowerComponents:AO3400A
- added Q6: AO3400A, SparkFun-DiscreteSemi:MOSFET-NCH-BSS138
- added R28: 330R, resistor:R-EU_R0402
- added R29: 10K, resistor:R-EU_R0402
- added U3: HY2213, PowerComponents:HY2213
- added U4: BQ24650, PowerComponents:BQ24650
- added U5: R5460X2XX, PowerComponents:R5460X2XX
- C1: value 2u2 -> 10u; device resistor:C-EUC0603 -> resistor:C-EUC1206
- C10, C14, C7: device resistor:C-EUC0603 -> resistor:C-EUC0402
- C11: value 22p -> 10u; device resistor:C-EUC0603 -> resistor:C-EUC1206
- C12: value 2u2 -> 100n; device resistor:C-EUC0603 -> resistor:C-EUC0402
- C13: value 100n -> 1u; device resistor:C-EUC0603 -> resistor:C-EUC0402
- C2, C3, C8: value 10u -> 100n; device resistor:C-EUC1210 -> resistor:C-EUC0402
- C4: value 1u -> 100n; device resistor:C-EUC0603 -> resistor:C-EUC0402
- C5: value 1u -> 10u; device resistor:C-EUC0603 -> resistor:C-EUC1206
- C6: value 100n -> 4u7; device resistor:C-EUC0603 -> resistor:C-EUC1206
- C9: value 4u7 -> 22p; device resistor:C-EUC1210 -> resistor:C-EUC0402
- D2: value 700mA/40V/533mV -> BAS70-04
- JP1: device pinhead:PINHD-1X10 -> pinhead:PINHD-1X3
- L1: device PowerComponents:INDUCTOR-DG6050 -> PowerComponents:INDUCTORMWSA1205
- Q1: value DMN6040SSD-13 -> FS8205; device transistor-power:IRF8313P -> PowerComponents:FS8205
- Q2: value DMN6040SSD-13 -> AO3400A; device transistor-power:IRF8313P -> PowerComponents:AO3400A
- Q3: value 220mA/50V/3.5Ω -> AO3400A; device SparkFun-DiscreteSemi:MOSFET-NCH-BSS138 -> PowerComponents:AO3400A
- R1: value 2R -> 5K1; device resistor:R-EU_R0603 -> resistor:R-EU_R0402
- R10: value 10R -> 4R7
- R11: value 40m -> 20K; device resistor:R-EU_R2512 -> resistor:R-EU_R0402
- R12: value 100K -> 300K; device resistor:R-EU_R0603 -> resistor:R-EU_R0402
- R13, R19, R20, R21, R26: device resistor:R-EU_R0603 -> resistor:R-EU_R0402
- R14: value 10K -> 2R; device resistor:R-EU_R0603 -> resistor:R-EU_R1206
- R15: value 10K -> 1K5; device resistor:R-EU_R0603 -> resistor:R-EU_R0402
- R16: value 300K -> 10K
- R17: value 2m -> 82K; device resistor:R-EU_R2512 -> resistor:R-EU_R0603
- R18: value 100R -> 1K; device resistor:R-EU_R0603 -> resistor:R-EU_R0402
- R2: value (none) -> 5K1; device resistor:R-EU_R0603 -> resistor:R-EU_R0402
- R22: value 10M -> 10K; device resistor:R-EU_R0603 -> resistor:R-EU_R0402
- R23: value 5K1 -> 27K; device resistor:R-EU_R0603 -> resistor:R-EU_R0402
- R24: value 5K1 -> 4K7; device resistor:R-EU_R0603 -> resistor:R-EU_R0402
- R25: value 10M -> 330R; device resistor:R-EU_R0603 -> resistor:R-EU_R0402
- R27: value 5R -> 10K; device resistor:R-EU_R0603 -> resistor:R-EU_R0402
- R3: value (none) -> 100R; device resistor:R-EU_R0603 -> resistor:R-EU_R0402
- R4: value 232K -> 0R02; device resistor:R-EU_R0603 -> resistor:R-EU_R1206
- R5: value 15K -> 100R; device resistor:R-EU_R0603 -> resistor:R-EU_R0402
- R6: value 100R -> 0R016; device resistor:R-EU_R0603 -> resistor:R-EU_R1206
- R7: value 10K -> 100R; device resistor:R-EU_R0603 -> resistor:R-EU_R0402
- R8: value 5K1 -> 4R7; device resistor:R-EU_R0603 -> resistor:R-EU_R1206
- R9: value 5K1 -> 100K; device resistor:R-EU_R0603 -> resistor:R-EU_R0402
- U1: value BQ24650 -> HY2213; device PowerComponents:BQ24650 -> PowerComponents:HY2213; LCSC_PN (none) -> C113632; MFG_PN (none) -> HY2213-BB3A
- U2: value BQ28Z610 -> BQ34Z100-G1; device PowerComponents:BQ28Z610 -> PowerComponents:BQ34Z100-G1; LCSC_PN (none) -> C91302; MFG_PN (none) -> BQ34Z100PWR-G1
Connections:
- removed net BAT: J1.BAT, Q2B.S, R25.2, R27.1, TP4.TP
- removed net CHG_GATE: R24.1, U2.CHG
- removed net DSG_GATE: R23.1, U2.DSG
- removed net N$32: C13.1, C14.1, R26.2, U2.VC1
- removed net N$33: C14.2, R27.2, U2.VC2
- removed net N$34: C12.1, U2.PBI
- removed net N$37: C10.1, R13.1, U2.SRN
- removed net N$39: C10.2, R18.1, U2.SRP
- new net N$13: Q3.G, U1.OUT
- new net N$15: Q3.D, R8.1
- new net N$16: R16.2, R17.1, U2.BAT
- new net N$2: Q5.G, U3.OUT
- new net N$20: C10.1, R13.1, U3.VDD
- new net N$21: C7.1, R7.1, U1.VDD
- new net N$22: R18.1, U5.V-
- new net N$23: C19.1, R25.2, U5.VC
- new net N$24: C20.1, R28.1, U5.VDD
- new net N$27: Q1.G2, U5.DOUT
- new net N$29: C2.1, C3.2, R3.2, U2.SRP
- new net N$30: C12.1, U2.REGIN
- new net REG25: C13.1, JP1.2, U2.REG25
- new net STAT_LED_EN: JP3.5, STAT1.A, STAT2.A
- net !BAT_CE!: now also JP3.3, R26.1; no longer JP1.4, R6.1
- net +3V3: now also JP2.1, R1.2, R2.2; no longer JP1.1, R8.2, R9.2, STAT1.A, STAT2.A
- net AGND: now also C12.2, C13.2, C14.2, Q6.S, R15.1, R16.1, R20.1, R23.1, R9.1, U2.P1, U2.P2, U2.P5/HDQ, U2.VEN, U2.VSS; no longer C4.2, Q3.S, R12.1, R3.1, R5.1, R7.1, TS.1, TS.3
- net BAL: now also BAL.TP, C10.2, Q5.S, R25.1, R7.2, R8.2, U3.VSS; no longer R26.1, TP5.TP
- net GND: now also C11.2, C15.2, C18.2, C3.1, C4.1, C6.2, H2.MOUNT, JP3.10, JP3.6, JP3.7, JP3.8, JP3.9, P-.TP, Q2.S, R22.1, R29.1, R3.1, R4.1, U4.PGND, U4.THERM; no longer C12.2, C13.2, C2.2, C3.2, C8.2, C9.2, JP2.10, JP2.5, JP2.6, JP2.7, JP2.8, JP2.9, Q1B.S, R14.1, R15.1, R17.2, R18.2, TP1.TP, U1.PGND, U1.THERM, U2.THERM, U2.VSS
- net MPPSET: now also Q6.D, R11.1, R15.2, U4.MPPSET; no longer Q3.D, R4.1, R5.2, U1.MPPSET
- net N$1: now also C18.1, R14.1; no longer C1.1, R1.1
- net N$10: now also C17.1, U4.BTST; no longer C7.1, U1.BTST
- net N$11: now also C15.1, U4.REGN; no longer C5.1, U1.REGN
- net N$12: now also C9.2, R12.1, R9.2, U4.VFB; no longer C11.2, R12.2, R16.1, U1.VFB
- net N$14: now also R21.1; no longer R20.1
- net N$18: now also Q5.D, R10.1; no longer R19.1, U2.PACK
- net N$25: now also C16.1, Q1.S1, R18.2, R4.2, R5.1; no longer Q2A.D, Q2B.D
- net N$26: now also Q1.G1, U5.COUT; no longer Q2A.G, R22.1, R23.2
- net N$28: now also C2.2, C4.2, R5.2, U2.SRN; no longer Q2B.G, R24.2, R25.1
- net N$3: now also R19.2, U4.VCC; no longer R10.2, U1.VCC
- net N$4: now also C11.1, C5.1, Q4.D, R11.2, R19.1; no longer C2.1, C3.1, Q1A.D, R10.1, R4.2
- net N$47: now also R27.1; no longer R21.1
- net N$5: now also Q4.G, U4.HIDRV; no longer Q1A.G, U1.HIDRV
- net N$6: now also C17.2, Q2.D, Q4.S, U4.PH; no longer C7.2, Q1A.S, Q1B.D, U1.PH
- net N$7: now also Q2.G, U4.LODRV; no longer Q1B.G, U1.LODRV
- net N$8: now also Q6.G, R20.2, R26.2; no longer Q3.G, R6.2, R7.2
- net N$81: now also R29.2; no longer R14.2
- net N$83: now also R22.2; no longer R15.2
- net N$9: now also C8.1, R6.1, U4.SRP; no longer C6.1, R11.1, U1.SRP
- net PANEL: now also JP3.4, P+.TP, R14.2; no longer JP2.3, R1.2, TP2.TP
- net RET: now also C16.2, C19.2, C20.2, C7.2, Q1.S2, Q3.S, RET.TP, U1.VSS, U5.VSS; no longer R13.2, R17.1, TP3.TP
- net SCL: now also JP2.3, R2.1, U2.P4/SCL; no longer JP2.2, R9.1, U2.SCL
- net SDA: now also JP2.2, R1.1, U2.P3/SDA; no longer JP2.1, R8.1, U2.SDA
- net STAT1: now also JP3.1, R21.2, U4.STAT1; no longer JP1.2, R20.2, U1.STAT1
- net STAT2: now also JP3.2, R27.2, U4.STAT2; no longer JP1.3, R21.2, U1.STAT2
- net TS1: now also JP1.3, R23.2, R24.1, U4.TS; no longer R2.1, R3.2, TS.2, U1.TS
- net TS2: now also JP1.1, U2.P6/TS; no longer TS.4, U2.TS1
- net VBAT: now also BAT.TP, C1.1, C6.1, C8.2, J1.BAT, JP2.10, JP2.5, JP2.6, JP2.7, JP2.8, JP2.9, R10.2, R12.2, R13.2, R17.2, R28.2, R6.2, U4.SRN; no longer C11.1, C6.2, C8.1, JP1.10, JP1.5, JP1.6, JP1.7, JP1.8, JP1.9, Q2A.S, R11.2, R16.2, R19.2, R22.2, U1.SRN
- net VREF: now also C14.1, R24.2, U4.TERM_EN, U4.VREF; no longer C4.1, R2.2, U1.TERM_EN, U1.VREF
Other:
- moved on the sheet: BAT_LED, C1, C10, C11, C12, C13, C14, C2, C3, C4, C5, C6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
